Commit message: the latest code with four leg of the dog

File: catkin_ws/src/smart_car/urdf/test_robot.urdf (robot description, URDF)
Before this commit: robot mycar, 2 links, 1 joints
Links:
- added link leftfront_link; visual box size=0.1 0.05 0.2
- added link rightback_link; visual box size=0.1 0.05 0.2
- added link rightfront_link; visual box size=0.1 0.05 0.2
Joints:
- added joint leftfront_joint: type continuous, parent base_link, child leftfront_link, origin xyz=2 1 0 rpy=0 0 0, axis -1 0 0
- added joint rightback_joint: type continuous, parent base_link, child rightback_link, origin xyz=-2 -1 0 rpy=0 1.5077 0, axis -1 0 0
- added joint rightfront_joint: type continuous, parent base_link, child rightfront_link, origin xyz=2 -1 0 rpy=0 1.5077 0, axis -1 0 0
- joint leftback_joint: axis -1 0 0 -> 1 0 0; origin xyz=0 0 0.05 rpy=1.5708 1.5708 0 -> xyz=-2 1 0 rpy=0 0 0
